File: wheatstone_bridge_board.brd (EAGLE design)
At the start: 64.5 x 93.7 mm, 66 parts

Commit message: rev 0.1
Parts:
- moved JP1 0.25 mm to (44.6, 93.0)
- moved JP2 0.25 mm to (16.1, 93.0)
Routing:
- added copper zone on layer 2, net GND
- removed copper zone on layer 2, net SIG
Other:
- board text added: "Wheatstone Bridge Board Hitzmann 2020"
