File: control_board.sch (EAGLE design)
At the start: 132 parts, among them J17 JST_PH_B3B-PH-K-S(LF)(SN), J18 JST_PH_B3B-PH-K-S(LF)(SN), J19 JST_PH_B3B-PH-K-S(LF)(SN), J20 JST_PH_B3B-PH-K-S(LF)(SN), J21 JST_PH_B3B-PH-K-S(LF)(SN), J22 JST_PH_B3B-PH-K-S(LF)(SN), J23 JST_PH_B3B-PH-K-S(LF)(SN), J24 JST_PH_B3B-PH-K-S(LF)(SN), J25 JST_PH_B3B-PH-K-S(LF)(SN), J26 JST_PH_B3B-PH-K-S(LF)(SN), J27 JST_PH_B3B-PH-K-S(LF)(SN), J28 JST_PH_B3B-PH-K-S(LF)(SN), J29 JST_PH_B3B-PH-K-S(LF)(SN), J30 JST_PH_B3B-PH-K-S(LF)(SN), J31 JST_PH_B3B-PH-K-S(LF)(SN), J32 JST_PH_B3B-PH-K-S(LF)(SN), J49 B4B-PH-K-S(LF)(SN), J50 B4B-PH-K-S(LF)(SN), J51 B4B-PH-K-S(LF)(SN), J52 B4B-PH-K-S(LF)(SN), J53 B4B-PH-K-S(LF)(SN), J54 B4B-PH-K-S(LF)(SN), J55 B4B-PH-K-S(LF)(SN), J56 B4B-PH-K-S(LF)(SN), J57 B4B-PH-K-S(LF)(SN), J58 B4B-PH-K-S(LF)(SN), J59 B4B-PH-K-S(LF)(SN), J60 B4B-PH-K-S(LF)(SN), J61 B4B-PH-K-S(LF)(SN), J62 B4B-PH-K-S(LF)(SN), J63 B4B-PH-K-S(LF)(SN), J64 B4B-PH-K-S(LF)(SN), Q1 BCF29SMD, U18 AD7730BRUZ, U19 AD5360BSTZ, U2 AMP-5103309-7-34PIN_5103309-7, U20 ADR425ARZ, U21 AD7730BRUZ, U23 AD7730BRUZ, U24 AD7730BRUZ, U25 AD7730BRUZ, U26 AD7730BRUZ, U27 AD7730BRUZ, U28 AD7730BRUZ, U4 ADR421ARZ, U5 AD7616BSTZ, X1 22-23-2031, Y1 KC2520B-C1, Y3 KC2520B-C1

Commit message: added GND to Teensy
Connections:
- net GND: now also U$1.GND1, U$1.GND3, U$1.GND6
Changed lines of the file:
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@@
 <part name="JP13" library="pinhead-2" deviceset="PINHD-2X12" device="_2.54-SMD"/>
 <part name="GND47" library="supply1" library_urn="urn:adsk.eagle:library:371" deviceset="GND" device=""/>
+<part name="GND50" library="supply1" library_urn="urn:adsk.eagle:library:371" deviceset="GND" device=""/>
 </parts>
 <sheets>
@@
 <attribute name="VALUE" x="-182.88" y="185.42" size="1.778" layer="96"/>
 </instance>
+<instance part="GND50" gate="1" x="-162.56" y="-22.86" smashed="yes">
+<attribute name="VALUE" x="-165.1" y="-25.4" size="1.778" layer="96"/>
+</instance>
 </instances>
 <busses>
@@
 <pinref part="GND47" gate="1" pin="GND"/>
 </segment>
+<segment>
+<pinref part="U$1" gate="G$1" pin="GND1"/>
+<wire x1="-162.56" y1="-5.08" x2="-162.56" y2="-15.24" width="0.1524" layer="91"/>
+<pinref part="U$1" gate="G$1" pin="GND3"/>
+<wire x1="-162.56" y1="-15.24" x2="-162.56" y2="-20.32" width="0.1524" layer="91"/>
+<wire x1="-157.48" y1="-5.08" x2="-157.48" y2="-15.24" width="0.1524" layer="91"/>
+<wire x1="-157.48" y1="-15.24" x2="-162.56" y2="-15.24" width="0.1524" layer="91"/>
+<junction x="-162.56" y="-15.24"/>
+<pinref part="U$1" gate="G$1" pin="GND6"/>
+<wire x1="-149.86" y1="-5.08" x2="-149.86" y2="-15.24" width="0.1524" layer="91"/>
+<wire x1="-149.86" y1="-15.24" x2="-157.48" y2="-15.24" width="0.1524" layer="91"/>
+<junction x="-157.48" y="-15.24"/>
+<pinref part="GND50" gate="1" pin="GND"/>
+</segment>
 </net>

Commit message: added caps and logo to control board
Parts:
- removed JP1: (no value), jumper:JP1Q
- added C12, C13, C14, C15, C16, C8: 100uF, rcl:CPOL-EUE3.5-8
Connections:
- removed net RPI_PWR: JP1.2, SV1.2, SV1.4
- removed net TEENSY_VIN: JP9.1, U$1.VIN
- new net PWR: C15.+, JP9.1, SV1.2, SV1.4, U$1.VIN
- net +5V: now also C13.+; no longer JP1.1
- net DVCC: now also C14.+
- net GND: now also C12.-, C13.-, C14.-, C15.-, C16.+, C8.-
- net VDD: now also C12.+, C8.+
- net VSS: now also C16.-
