File: electronics/dual/control_board.brd (EAGLE design)
At the start: 190 x 180 mm, 136 parts, among them J17 JST_PH_B3B-PH-K-S(LF)(SN), J18 JST_PH_B3B-PH-K-S(LF)(SN), J19 JST_PH_B3B-PH-K-S(LF)(SN), J20 JST_PH_B3B-PH-K-S(LF)(SN), J21 JST_PH_B3B-PH-K-S(LF)(SN), J22 JST_PH_B3B-PH-K-S(LF)(SN), J23 JST_PH_B3B-PH-K-S(LF)(SN), J24 JST_PH_B3B-PH-K-S(LF)(SN), J25 JST_PH_B3B-PH-K-S(LF)(SN), J26 JST_PH_B3B-PH-K-S(LF)(SN), J27 JST_PH_B3B-PH-K-S(LF)(SN), J28 JST_PH_B3B-PH-K-S(LF)(SN), J29 JST_PH_B3B-PH-K-S(LF)(SN), J30 JST_PH_B3B-PH-K-S(LF)(SN), J31 JST_PH_B3B-PH-K-S(LF)(SN), J32 JST_PH_B3B-PH-K-S(LF)(SN), U18 AD7730BRUZ, U19 AD5360BSTZ, U20 ADR425ARZ, U21 AD7730BRUZ, U23 AD7730BRUZ, U24 AD7730BRUZ, U25 AD7730BRUZ, U26 AD7730BRUZ, U27 AD7730BRUZ, U28 AD7730BRUZ, U4 ADR421ARZ, U5 AD7616BSTZ, X1 22-23-2031, Y1 KC2520B-C1, Y3 KC2520B-C1

Commit message: added raspi firmware
Parts:
- added SV1: (no value), con-lsta:FE20-2
- moved LED1 38.4 mm to (12.3, 141.1), turned to 90 degrees
- moved R11 31.4 mm to (17.6, 141.1), turned to 0 degrees
Connections:
- new net 3_3V: SV1.17
- new net N$12: SV1.28
- new net N$13: SV1.27
- net ADC_2_CONVST: now also SV1.5
- net GND: now also SV1.14, SV1.20, SV1.25, SV1.30, SV1.34, SV1.39, SV1.6, SV1.9
- net HEARTBEAT: now also SV1.3
- net LC_1_CS0: now also SV1.29
- net LC_1_CS1: now also SV1.26
- net LC_1_CS2: now also SV1.24
- net LC_1_CS3: now also SV1.22
- net LC_1_CS4: now also SV1.40
- net LC_1_CS5: now also SV1.38
- net LC_1_CS6: now also SV1.37
- net LC_1_CS7: now also SV1.36
- net LC_1_RDY0: now also SV1.13
- net LC_1_RDY1: now also SV1.15
- net LC_1_RDY2: now also SV1.16
- net LC_1_RDY3: now also SV1.18
- net LC_1_RDY4: now also SV1.31
- net LC_1_RDY5: now also SV1.32
- net LC_1_RDY6: now also SV1.33
- net LC_1_RDY7: now also SV1.35
- net LDAC: now also SV1.11
- net MISO: now also SV1.21
- net MOSI: now also SV1.19
- net PWR: now also SV1.2, SV1.4
- net RX: now also SV1.10
- net SCLK: now also SV1.23
- net SS_ADC_2: now also SV1.7
- net SS_DAC_2: now also SV1.12
- net TX: now also SV1.8
Routing:
- net TX: track 13.2 -> 70.8 mm
- net RX: track 13.2 -> 66.4 mm
- net SS_DAC_2: track 189.1 -> 227.7 mm
- net MOSI: track 327.6 -> 365.7 mm
- net MISO: track 348.0 -> 386.1 mm
- net HEARTBEAT: track 7.08 -> 43.1 mm
- net SS_ADC_2: track 72.4 -> 108.4 mm
- net LDAC: track 173.1 -> 209.1 mm
- net ADC_2_CONVST: track 75.8 -> 111.8 mm
- net LC_1_CS5: track 54.7 -> 81.1 mm
- net LC_1_CS4: track 62.5 -> 88.9 mm
- net LC_1_CS7: track 44.3 -> 69.8 mm
- net LC_1_RDY5: track 90.1 -> 114.4 mm
- net LC_1_CS1: track 134.6 -> 157.9 mm
- net LC_1_CS2: track 124.4 -> 147.8 mm
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